File: board/6502ino.sch (KiCad schematic (older format))
At the start: 17 parts, among them U1 W65C02S, U2 IDT71256SA, U3 74HC165, U4 74HC595, U5 74AC00

Commit message: Reduce number of ICs to 3, first working arduino sketch
Parts:
- removed C4, C5: 100nF, Capacitor_THT:C_Disc_D3.0mm_W1.6mm_P2.50mm, symbol Device:C_Small
- removed R1: 1k, Resistor_THT:R_Axial_DIN0207_L6.3mm_D2.5mm_P7.62mm_Horizontal, symbol Device:R
- removed U3: 74HC165, Package_DIP:DIP-16_W7.62mm_Socket, symbol 74xx:74LS165
- removed U4: 74HC595, Package_DIP:DIP-16_W7.62mm_Socket, symbol 74xx:74HCT595
- removed unit 4 of U5
- added R1, R10, R2, R3, R4, R5, R6, R7, R8, R9: 6K8, Resistor_THT:R_Axial_DIN0207_L6.3mm_D2.5mm_P7.62mm_Horizontal, symbol Device:R_Small
- added R12: 100, Resistor_THT:R_Axial_DIN0207_L6.3mm_D2.5mm_P7.62mm_Horizontal, symbol Device:R_Small
- added unit 4 of U3
- C4: renamed from C10; footprint Capacitor_THT:C_Disc_D3.0mm_W1.6mm_P2.50mm -> Capacitor_THT:C_Disc_D4.3mm_W1.9mm_P5.00mm
- R11: renamed from R2; value 10k -> 6k8
- renumbered U5 to U3
Connections:
- net labels removed: IOIN, IOOUT, PHI1, RDY
- wire segments 140 -> 121
- no-connect marks 29 -> 21
Other:
- note removed: "(INPUT BUFFER)"
- note removed: "(OUTPUT BUFFER)"
- moved on the sheet: U3A, U3B, U3C, U3E

Commit message: Fiddling with the layout
Other:
- moved on the sheet: U3B, U3D
Changed lines of the file:
@@
 L 74xx:74HC00 U3
 U 2 1 5D868474
-P 2400 1950
-F 0 "U3" H 2400 2275 50  0000 C CNN
-F 1 "74AC00" H 2400 2184 50  0000 C CNN
-F 2 "Package_DIP:DIP-14_W7.62mm_Socket" H 2400 1950 50  0001 C CNN
-F 3 "http://www.ti.com/lit/gpn/sn74hc00" H 2400 1950 50  0001 C CNN
-	2    2400 1950
+P 6400 3350
+F 0 "U3" H 6400 3675 50  0000 C CNN
+F 1 "74AC00" H 6400 3584 50  0000 C CNN
+F 2 "Package_DIP:DIP-14_W7.62mm_Socket" H 6400 3350 50  0001 C CNN
+F 3 "http://www.ti.com/lit/gpn/sn74hc00" H 6400 3350 50  0001 C CNN
+	2    6400 3350
 	1    0    0    -1
 $EndComp
@@
 D7
 Text Label 8750 2250 0    50   ~ 0
-D6
+D5
 Text Label 8750 2150 0    50   ~ 0
-D4
+D3
 Text Label 8750 2050 0    50   ~ 0
-D2
+D1
 Text Label 8750 1950 0    50   ~ 0
 D0
 Text Label 8750 1850 0    50   ~ 0
-D1
+D2
 Text Label 8750 1750 0    50   ~ 0
-D3
+D4
 Text Label 8750 1650 0    50   ~ 0
-D5
+D6
 Wire Wire Line
 	8650 1650 8750 1650
@@
 	8650 2350 8750 2350
 Text Label 7350 3050 2    50   ~ 0
+A0
+Text Label 7350 2950 2    50   ~ 0
+A1
+Text Label 7350 2850 2    50   ~ 0
 A2
-Text Label 7350 2950 2    50   ~ 0
-A3
-Text Label 7350 2850 2    50   ~ 0
+Text Label 7350 2750 2    50   ~ 0
 A4
-Text Label 7350 2750 2    50   ~ 0
+Text Label 7350 2650 2    50   ~ 0
 A5
-Text Label 7350 2650 2    50   ~ 0
-A6
 Text Label 7350 2550 2    50   ~ 0
 A7
 Text Label 7350 2450 2    50   ~ 0
-A8
+A14
 Text Label 7350 2350 2    50   ~ 0
-A9
+A13
 Text Label 7350 2250 2    50   ~ 0
-A10
+A12
 Text Label 7350 2150 2    50   ~ 0
 A11
 Text Label 7350 2050 2    50   ~ 0
-A12
+A10
 Text Label 7350 1950 2    50   ~ 0
-A13
+A9
 Text Label 7350 1850 2    50   ~ 0
-A14
+A8
 Text Label 7350 1750 2    50   ~ 0
-A1
+A6
 Text Label 7350 1650 2    50   ~ 0
-A0
+A3
 Wire Wire Line
 	7350 1650 7450 1650
@@
 Wire Wire Line
 	4500 6850 4450 6850
-NoConn ~ 4500 6950
 $Comp
 L 74xx:7400 U3
 U 4 1 5D830640
-P 6400 3350
-F 0 "U3" H 6400 3675 50  0000 C CNN
-F 1 "74AC00" H 6400 3584 50  0000 C CNN
-F 2 "Package_DIP:DIP-14_W7.62mm_Socket" H 6400 3350 50  0001 C CNN
-F 3 "http://www.ti.com/lit/gpn/sn7400" H 6400 3350 50  0001 C CNN
-	4    6400 3350
+P 2400 1950
+F 0 "U3" H 2400 2275 50  0000 C CNN
+F 1 "74AC00" H 2400 2184 50  0000 C CNN
+F 2 "Package_DIP:DIP-14_W7.62mm_Socket" H 2400 1950 50  0001 C CNN
+F 3 "http://www.ti.com/lit/gpn/sn7400" H 2400 1950 50  0001 C CNN
+	4    2400 1950
 	1    0    0    -1
 $EndComp
@@
 L Device:R_Small R9
 U 1 1 5D8652E0
+P 4150 7150
+F 0 "R9" V 4100 7000 50  0000 C CNN
+F 1 "6K8" V 4100 7350 50  0000 C CNN
+F 2 "Resistor_THT:R_Axial_DIN0207_L6.3mm_D2.5mm_P7.62mm_Horizontal" H 4150 7150 50  0001 C CNN
+F 3 "~" H 4150 7150 50  0001 C CNN
+	1    4150 7150
+	0    -1   1    0
+$EndComp
+Text Label 3800 7150 2    50   ~ 0
+D7
+Wire Wire Line
+	4050 7150 3800 7150
+Wire Wire Line
+	4500 7150 4250 7150
+$Comp
+L Device:R_Small R10
+U 1 1 5D8652E9
 P 4150 7250
-F 0 "R9" V 4100 7100 50  0000 C CNN
+F 0 "R10" V 4100 7100 50  0000 C CNN
 F 1 "6K8" V 4100 7450 50  0000 C CNN
 F 2 "Resistor_THT:R_Axial_DIN0207_L6.3mm_D2.5mm_P7.62mm_Horizontal" H 4150 7250 50  0001 C CNN
@@
 $EndComp
 Text Label 3800 7250 2    50   ~ 0
-D7
+D6
 Wire Wire Line
 	4050 7250 3800 7250
 Wire Wire Line
 	4500 7250 4250 7250
-$Comp
-L Device:R_Small R10
-U 1 1 5D8652E9
-P 4150 7350
-F 0 "R10" V 4100 7200 50  0000 C CNN
-F 1 "6K8" V 4100 7550 50  0000 C CNN
-F 2 "Resistor_THT:R_Axial_DIN0207_L6.3mm_D2.5mm_P7.62mm_Horizontal" H 4150 7350 50  0001 C CNN
-F 3 "~" H 4150 7350 50  0001 C CNN
-	1    4150 7350
-	0    -1   1    0
-$EndComp
-Text Label 3800 7350 2    50   ~ 0
-D6
-Wire Wire Line
-	4050 7350 3800 7350
-Wire Wire Line
-	4500 7350 4250 7350
 $Comp
 L Device:R_Small R8
 U 1 1 5D880461
-P 4150 7150
-F 0 "R8" V 4100 7000 50  0000 C CNN
-F 1 "6K8" V 4100 7350 50  0000 C CNN
-F 2 "Resistor_THT:R_Axial_DIN0207_L6.3mm_D2.5mm_P7.62mm_Horizontal" H 4150 7150 50  0001 C CNN
-F 3 "~" H 4150 7150 50  0001 C CNN
-	1    4150 7150
-	0    -1   1    0
-$EndComp
-Text Label 3800 7150 2    50   ~ 0
-IOSELECT
-Wire Wire Line
-	4500 7150 4250 7150
-$Comp
-L Device:R_Small R7
-U 1 1 5D8872E8
 P 4150 7050
-F 0 "R7" V 4100 6900 50  0000 C CNN
+F 0 "R8" V 4100 6900 50  0000 C CNN
 F 1 "6K8" V 4100 7250 50  0000 C CNN
 F 2 "Resistor_THT:R_Axial_DIN0207_L6.3mm_D2.5mm_P7.62mm_Horizontal" H 4150 7050 50  0001 C CNN
@@
 $EndComp
 Text Label 3800 7050 2    50   ~ 0
+IOSELECT
+Wire Wire Line
+	4500 7050 4250 7050
+$Comp
+L Device:R_Small R7
+U 1 1 5D8872E8
+P 4150 6950
+F 0 "R7" V 4100 6800 50  0000 C CNN
+F 1 "6K8" V 4100 7150 50  0000 C CNN
+F 2 "Resistor_THT:R_Axial_DIN0207_L6.3mm_D2.5mm_P7.62mm_Horizontal" H 4150 6950 50  0001 C CNN
+F 3 "~" H 4150 6950 50  0001 C CNN
+	1    4150 6950
+	0    -1   1    0
+$EndComp
+Text Label 3800 6950 2    50   ~ 0
 RWB
 Wire Wire Line
+	4050 6950 3800 6950
+Wire Wire Line
+	4500 6950 4250 6950
+Wire Wire Line
 	4050 7050 3800 7050
-Wire Wire Line
-	4500 7050 4250 7050
-Wire Wire Line
-	4050 7150 3800 7150
 $Comp
 L Device:R_Small R12
@@
 	7450 3350 6700 3350
 NoConn ~ 3700 2050
+NoConn ~ 4500 7350
 $EndSCHEMATC

Commit message: Fix: Connect BE to +5V
Connections:
- wire segments 121 -> 122
- no-connect marks 21 -> 20
Changed lines of the file:
@@
 Title "6502ino"
 Date "2019-09-20"
-Rev "1"
+Rev "2"
 Comp ""
 Comment1 ""
@@
 Wire Wire Line
 	4500 2550 4600 2550
-NoConn ~ 4500 2250
 Text Label 4600 2150 0    50   ~ 0
 PHI2
@@
 NoConn ~ 3700 2050
 NoConn ~ 4500 7350
+$Comp
+L power:+5V #PWR?
+U 1 1 5D96B089
+P 4650 2250
+F 0 "#PWR?" H 4650 2100 50  0001 C CNN
+F 1 "+5V" V 4665 2378 50  0000 L CNN
+F 2 "" H 4650 2250 50  0001 C CNN
+F 3 "" H 4650 2250 50  0001 C CNN
+	1    4650 2250
+	0    1    1    0
+$EndComp
+Wire Wire Line
+	4500 2250 4650 2250
 $EndSCHEMATC
